Commit message: Fix: Updated AMR to differential drive with rear caster wheel

File: amr_ws/src/amr_description/urdf/amr.urdf (robot description, URDF)
Before this commit: robot amr_robot, 2 links, 1 joints
Links:
- removed link caster_wheel
- added link caster_wheel_rear; visual sphere radius=0.1
- added link wheel_front_left; visual cylinder length=0.04 radius=0.1
- added link wheel_front_right; visual cylinder length=0.04 radius=0.1
Joints:
- removed joint base_to_caster
- added joint joint_caster_wheel_rear: type fixed, parent base_link, child caster_wheel_rear, origin xyz=-0.2 0 0 rpy=0 0 0
- added joint joint_wheel_front_left: type continuous, parent base_link, child wheel_front_left, origin xyz=0.2 0.15 0 rpy=1.57 0 0, axis 0 0 1
- added joint joint_wheel_front_right: type continuous, parent base_link, child wheel_front_right, origin xyz=0.2 -0.15 0 rpy=1.57 0 0, axis 0 0 1
